File: PowerBoard1AMp.sch (EAGLE design)
At the start: 4 parts, among them IC1 VREG

Commit message: Added two capacitors for regulators
Parts:
- added C1, C2: 10uF, fablab:UNPOLARIZED_CAPACITOR1206
Connections:
- net GND: now also C1.1, C2.1
- net N$2: now also C2.2
- net N$4: now also C1.2
Changed lines of the file:
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@@
 <?xml version="1.0" encoding="utf-8"?>
 <!DOCTYPE eagle SYSTEM "eagle.dtd">
-<eagle version="6.3">
+<eagle version="7.3.0">
 <drawing>
 <settings>
@@
 <layer number="97" name="Info" color="7" fill="1" visible="yes" active="yes"/>
 <layer number="98" name="Guide" color="6" fill="1" visible="yes" active="yes"/>
+<layer number="99" name="SpiceOrder" color="7" fill="1" visible="yes" active="yes"/>
 <layer number="100" name="Muster" color="7" fill="1" visible="no" active="no"/>
 <layer number="101" name="Patch_Top" color="12" fill="4" visible="no" active="yes"/>
@@
 <layer number="111" name="LPC17xx" color="7" fill="1" visible="no" active="yes"/>
 <layer number="112" name="tSilk" color="7" fill="1" visible="yes" active="yes"/>
+<layer number="113" name="IDFDebug" color="4" fill="1" visible="yes" active="yes"/>
 <layer number="116" name="Patch_BOT" color="9" fill="4" visible="no" active="yes"/>
 <layer number="121" name="_tsilk" color="7" fill="1" visible="no" active="yes"/>
@@
 <part name="U$1" library="ng" deviceset="GND" device=""/>
 <part name="U$2" library="ng" deviceset="SIGNAL" device=""/>
+<part name="C1" library="fablab" deviceset="UNPOLARIZED_CAPACITOR" device="1206" value="10uF"/>
+<part name="C2" library="fablab" deviceset="UNPOLARIZED_CAPACITOR" device="1206" value="10uF"/>
 </parts>
 <sheets>
@@
 <instance part="U$1" gate="G$1" x="10.16" y="30.48"/>
 <instance part="U$2" gate="G$1" x="12.7" y="45.72" rot="R90"/>
+<instance part="C1" gate="1" x="17.78" y="40.64" rot="R90"/>
+<instance part="C2" gate="1" x="45.72" y="38.1" rot="R90"/>
 </instances>
 <busses>
@@
 <wire x1="27.94" y1="33.02" x2="27.94" y2="30.48" width="0.1524" layer="91"/>
 <wire x1="10.16" y1="30.48" x2="10.16" y2="33.02" width="0.1524" layer="91"/>
-<wire x1="10.16" y1="33.02" x2="27.94" y2="33.02" width="0.1524" layer="91"/>
+<wire x1="10.16" y1="33.02" x2="17.78" y2="33.02" width="0.1524" layer="91"/>
 <junction x="27.94" y="33.02"/>
+<pinref part="C1" gate="1" pin="1"/>
+<wire x1="17.78" y1="33.02" x2="27.94" y2="33.02" width="0.1524" layer="91"/>
+<wire x1="17.78" y1="35.56" x2="17.78" y2="33.02" width="0.1524" layer="91"/>
+<junction x="17.78" y="33.02"/>
+<pinref part="C2" gate="1" pin="1"/>
+<wire x1="45.72" y1="33.02" x2="27.94" y2="33.02" width="0.1524" layer="91"/>
 </segment>
 <segment>
@@
 <pinref part="IC1" gate="G$1" pin="OUT@1"/>
 <pinref part="U$3" gate="G$1" pin="3"/>
-<wire x1="38.1" y1="43.18" x2="76.2" y2="43.18" width="0.1524" layer="91"/>
+<wire x1="38.1" y1="43.18" x2="45.72" y2="43.18" width="0.1524" layer="91"/>
+<pinref part="C2" gate="1" pin="2"/>
+<wire x1="45.72" y1="43.18" x2="76.2" y2="43.18" width="0.1524" layer="91"/>
+<wire x1="45.72" y1="40.64" x2="45.72" y2="43.18" width="0.1524" layer="91"/>
+<junction x="45.72" y="43.18"/>
 </segment>
 </net>
@@
 <pinref part="U$2" gate="G$1" pin="P$2"/>
 <pinref part="IC1" gate="G$1" pin="IN"/>
-<wire x1="12.7" y1="45.72" x2="20.32" y2="45.72" width="0.1524" layer="91"/>
-</segment>
-</net>
+<wire x1="12.7" y1="45.72" x2="17.78" y2="45.72" width="0.1524" layer="91"/>
+<pinref part="C1" gate="1" pin="2"/>
+<wire x1="17.78" y1="45.72" x2="20.32" y2="45.72" width="0.1524" layer="91"/>
+<wire x1="17.78" y1="43.18" x2="17.78" y2="45.72" width="0.1524" layer="91"/>
+<junction x="17.78" y="45.72"/>
+</segment>
+</net>

Commit message: Change the pins for VCC and GND in connector
Connections:
- removed net N$2: C2.2, IC1.OUT@1, U$3.3
- removed net RX: U$3.4
- removed net TX: U$3.2
- new net VCC: C2.2, IC1.OUT@1, U$3.2
- net GND: now also U$3.4; no longer U$3.1
Changed lines of the file:
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@@
 <instance part="IC1" gate="G$1" x="27.94" y="40.64"/>
 <instance part="GND1" gate="1" x="27.94" y="27.94"/>
-<instance part="GND2" gate="1" x="55.88" y="50.8"/>
+<instance part="GND2" gate="1" x="101.6" y="38.1"/>
 <instance part="U$1" gate="G$1" x="10.16" y="30.48"/>
 <instance part="U$2" gate="G$1" x="12.7" y="45.72" rot="R90"/>
@@
 </busses>
 <nets>
-<net name="TX" class="0">
-<segment>
-<pinref part="U$3" gate="G$1" pin="2"/>
-<wire x1="83.82" y1="45.72" x2="96.52" y2="45.72" width="0.1524" layer="91"/>
-<label x="91.44" y="45.72" size="1.778" layer="95"/>
-</segment>
-</net>
-<net name="RX" class="0">
-<segment>
-<pinref part="U$3" gate="G$1" pin="4"/>
-<wire x1="83.82" y1="43.18" x2="96.52" y2="43.18" width="0.1524" layer="91"/>
-<label x="91.44" y="43.18" size="1.778" layer="95"/>
-</segment>
-</net>
 <net name="GND" class="0">
 <segment>
@@
 </segment>
 <segment>
-<pinref part="U$3" gate="G$1" pin="1"/>
-<wire x1="76.2" y1="45.72" x2="60.96" y2="45.72" width="0.1524" layer="91"/>
-<wire x1="60.96" y1="45.72" x2="60.96" y2="55.88" width="0.1524" layer="91"/>
-<wire x1="60.96" y1="55.88" x2="55.88" y2="55.88" width="0.1524" layer="91"/>
 <pinref part="GND2" gate="1" pin="GND"/>
-<wire x1="55.88" y1="55.88" x2="55.88" y2="53.34" width="0.1524" layer="91"/>
+<wire x1="101.6" y1="40.64" x2="101.6" y2="43.18" width="0.1524" layer="91"/>
+<pinref part="U$3" gate="G$1" pin="4"/>
+<wire x1="101.6" y1="43.18" x2="83.82" y2="43.18" width="0.1524" layer="91"/>
 </segment>
 </net>
-<net name="N$2" class="0">
+<net name="VCC" class="0">
 <segment>
 <pinref part="IC1" gate="G$1" pin="OUT@1"/>
-<pinref part="U$3" gate="G$1" pin="3"/>
 <wire x1="38.1" y1="43.18" x2="45.72" y2="43.18" width="0.1524" layer="91"/>
 <pinref part="C2" gate="1" pin="2"/>
-<wire x1="45.72" y1="43.18" x2="76.2" y2="43.18" width="0.1524" layer="91"/>
 <wire x1="45.72" y1="40.64" x2="45.72" y2="43.18" width="0.1524" layer="91"/>
-<junction x="45.72" y="43.18"/>
+<label x="40.64" y="43.18" size="1.778" layer="95"/>
+</segment>
+<segment>
+<pinref part="U$3" gate="G$1" pin="2"/>
+<wire x1="83.82" y1="45.72" x2="93.98" y2="45.72" width="0.1524" layer="91"/>
+<label x="88.9" y="45.72" size="1.778" layer="95"/>
 </segment>
 </net>
